File: circuits/handheld-1/hh-1.sch (KiCad schematic (older format))
At the start: 42 parts, among them SW1 SW_DPDT_x2, U1 TL074

Commit message: hh-1 schema nearly simulating
Parts:
- removed BT? (x2): Battery, symbol Device:Battery
- removed RV?: R_POT_US, symbol Device:R_POT_US
- removed SW1, SW?: SW_DPDT_x2, symbol Switch:SW_DPDT_x2
- added J1: Conn_01x01_Female, symbol Connector:Conn_01x01_Female
- added R10: 22k, symbol Device:R_US
- added R17: 100k, symbol Device:R_US
- C10: renamed from C?; value CP -> 10u
- C11: renamed from C?; value CP -> 1u
- C12, C13, C14: renamed from C?; value CP -> 100u
- C2, C3, C4, C5: renamed from C?; value C -> 100n
- C6, C7, C8, C9: renamed from C?; value C -> 47n
- LS1: renamed from LS?; value Speaker -> 8
- R11: renamed from R?; value R_US -> 1M
- R12: renamed from R?; value R_US -> 100k
- R13: renamed from R?; value R_US -> 1k5
- R14: renamed from R?; value R_US -> 10k
- R15, R16: renamed from R?; value R_US -> 8k2
- R4, R5: renamed from R?; value R_US -> 33k
- R6: renamed from R?; value R_US -> 15k
- R7, R8, R9: renamed from R?; value R_US -> 22k
- gave numbers to parts that had none: 6
Connections:
- net labels added: +9V, -9V
- wire segments 142 -> 143
Other:
- moved on the sheet: U1C
